File: ESP32_4_layer/User_Interface.kicad_sch (KiCad schematic)
At the start: 11 parts, among them J4 Conn_01x05_Pin, J5 Conn_01x04_Pin, Q2 BC817, Q3 BC817

Commit message: PCB Stack up, netlist and constrainsts applied
Signed-off-by: jayaraj <jayarajemengineer@gmail.com>
Parts:
- S1, S2: footprint USLPT2819DT2TR:SW_USLPT2819DT2TR -> Own_Library:SW_USLPT2819DT2TR
Changed lines of the file:
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@@
 			)
 		)
-		(property "Footprint" "USLPT2819DT2TR:SW_USLPT2819DT2TR"
+		(property "Footprint" "Own_Library:SW_USLPT2819DT2TR"
 			(at 234.95 68.58 0)
 			(effects
@@
 			)
 		)
-		(property "Footprint" "USLPT2819DT2TR:SW_USLPT2819DT2TR"
+		(property "Footprint" "Own_Library:SW_USLPT2819DT2TR"
 			(at 248.92 124.46 0)
 			(effects

Commit message: Routing finished_1
Connections:
- net SCL: now also J5.2 (Pin_2); no longer J5.3 (Pin_3)
- net SDA: now also J5.3 (Pin_3); no longer J5.2 (Pin_2)
Changed lines of the file:
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@@
 		)
 	)
-	(hierarchical_label "SCL"
+	(hierarchical_label "SDA"
 		(shape bidirectional)
 		(at 107.95 67.31 0)
@@
 		)
 	)
-	(hierarchical_label "SDA"
+	(hierarchical_label "SCL"
 		(shape bidirectional)
 		(at 107.95 64.77 0)
